Commit message: Updating repo with motor control and simple map demo

File: masbot_description/urdf/masbot.urdf (robot description, URDF)
Before this commit: robot masbot, 21 links, 20 joints
Links:
- removed link imu_link
Joints:
- removed joint imu_joint
- joint camera_joint: origin xyz=0 0 0.055 rpy=0 0 0 -> xyz=0 0 0.02 rpy=0 0 0
- joint lidar_joint: origin xyz=0 0 0.02 rpy=0 0 0 -> xyz=0 0 0.055 rpy=0 0 0

Commit message: pushing for thorough URDF/TF inspection

File: masbot_description/urdf/masbot.urdf (robot description, URDF)
Before this commit: robot masbot, 20 links, 19 joints
Links:
- removed link camera_link
- removed link ultrasonic_front_link
- removed link ultrasonic_left_link
- removed link ultrasonic_right_link
Joints:
- removed joint camera_joint
- removed joint ultrasonic_front_joint
- removed joint ultrasonic_left_joint
- removed joint ultrasonic_right_joint
